File: PTP_jakov_ozbolt_project-1/PTP_jakov_ozbolt_project-1.kicad_sch (KiCad schematic)
At the start: 2 parts

Commit message: LV3
Parts:
- removed R1, R2: R_Small, symbol Device:R_Small
- added C1: C, symbol Device:C
- added C2, C3: C_Polarized, symbol Device:C_Polarized
- added D1: D_Zener_Filled, symbol Device:D_Zener_Filled
- added J1: Screw_Terminal_01x02, symbol Connector:Screw_Terminal_01x02
- added L1: L, symbol Device:L
- added R1: R, symbol Device:R
- added SW1: SW_MEC_5G, symbol Switch:SW_MEC_5G
- added U1: LM2574N-5, Package_DIP:DIP-8_W7.62mm, symbol Regulator_Switching:LM2574N-5
- added U6: ~, symbol SN74LVC1G11:SN74LVC1G11
Connections:
- net GND: now also C1.1, J1.1 (Pin_1), SW1.1 (A), SW1.2 (A), U6.2 (GND)
- new net: C3.1, L1.2
- new net: D1.1 (K), L1.1, U1.7 (OUT)
- new net: R1.1, SW1.3 (B), SW1.4 (B)
- new net +5V: U6.5 (VCC)
- new net Clock: U6.3 (B)
- new net Q1: U6.6 (C)
- new net Q3: U6.1 (A)
- new net Reset: U6.4 (Y)
- new net VD: C2.1, J1.2 (Pin_2), U1.5 (VIN)
- no-connect marks 1 -> 0

Commit message: Update PTP_jakov_ozbolt_project-1.kicad_sch
Parts:
- added C4: 100n, symbol Device:C
- added C5: 10u, symbol Device:C
- added D1, D2, D3, D5: LED, symbol Device:LED
- added H1, H2, H3, H4: MountingHole, symbol Mechanical:MountingHole
- added R10, R11, R12, R15, R24, R9: 10k, symbol Device:R
- added R14, R16, R17, R18, R5, R6, R8: 2k, symbol Device:R
- added R21, R22: 47k, symbol Device:R
- added R25, R26, R27, R28: 4k7, symbol Device:R
- added SW4: ~, symbol Switch:SW_SPDT_312
- added U2, U3: 4027, symbol 4xxx:4027
- added U4: 74LS47, symbol 74xx:74LS47
- added U5: HDSP-7401, Display_7Segment:HDSP-7401, symbol Display_Character:HDSP-7401
- added U7: NE555P, Package_DIP:DIP-8_W7.62mm, symbol Timer:NE555P
- C1: renamed from C2; value C_Polarized -> 22u; footprint (none) -> Capacitor_THT:CP_Radial_D5.0mm_P2.00mm; Manifacturer (none) -> AISHI; Manifacturer part number (none) -> EWH1EM220D11OT
- C10: renamed from C3; value C_Polarized -> 220u
- C6: renamed from C1; value C -> 1u
- D4: renamed from D1; value D_Zener_Filled -> 11DQ06; footprint (none) -> Diode_THT:D_DO-41_SOD81_P12.70mm_Horizontal; Manifacturer (none) -> SMC DIODE SOLUTIONS
- J1: value Screw_Terminal_01x02 -> ~; footprint (none) -> TerminalBlock_MetzConnect:TerminalBlock_MetzConnect_Type011_RT05502HBLC_1x02_P5.00mm_Horizontal; Manifacture part number (none) -> DG301-5.0-02P-12-00A(H); Manifacturer (none) -> DEGSON ELECTRONICS
- L1: value L -> 330u
- R23: renamed from R1; value R -> 2k
- SW3: renamed from SW1; value SW_MEC_5G -> ~
- U1: footprint Package_DIP:DIP-8_W7.62mm -> Package_DIP:DIP-8_W7.62mm_Socket_LongPads; Manifacture part number (none) -> LM2574N-5G; Manufacture (none) -> ONSEMI
Connections:
- net +5V: now also C10.1, L1.2, U1.1 (FB), C4.1, R10.1, R11.1, R12.1, R15.1, R21.1, R24.2, R9.1, U2.16 (VDD), U3.16 (VDD), U4.16 (VCC), U5.1 (CA), U5.6 (CA), U7.4 (R), U7.8 (VCC)
- net Clock: now also R24.1, SW4.1 (B), U2.3 (C)
- net GND: now also C1.2, C10.2, D4.2 (A), U1.2 (SGND), U1.3 (~{ON}/OFF), U1.4 (PGND), C4.2, C5.2, R25.2, R26.2, R27.2, R28.2, U2.7 (S), U2.8 (VSS), U2.9 (S), U3.7 (S), U3.8 (VSS), U3.9 (S), U4.8 (GND), U7.1 (GND)
- net Q1: now also D2.2 (A), U2.15 (Q), U3.3 (C), U4.1 (B)
- net Q3: now also D5.2 (A), U3.15 (Q), U4.6 (D)
- net Reset: now also U2.12 (R), U2.4 (R), U3.12 (R), U3.4 (R)
- net at C6.2: now also R23.2, SW4.3 (A)
- new net: R11.2, U3.5 (K), U3.6 (J)
- new net: R15.2, U4.3 (LT), U4.4 (BI), U4.5 (RBI)
- new net: D3.1 (K), R27.1
- new net: R5.2, U5.10 (A)
- new net: R17.2, U5.2 (F)
- new net: R18.2, U5.3 (G)
- new net: R16.2, U5.4 (E)
- new net: R14.2, U5.5 (D)
- new net: R8.2, U5.8 (C)
- new net: R6.2, U5.9 (B)
- new net: D2.1 (K), R26.1
- new net: R14.1, U4.10 (d)
- new net: R8.1, U4.11 (c)
- new net: R6.1, U4.12 (b)
- new net: R5.1, U4.13 (a)
- new net: R18.1, U4.14 (g)
- new net: R17.1, U4.15 (f)
- new net: R16.1, U4.9 (e)
- new net: C5.1, R22.2, U7.2 (TR), U7.6 (THR)
- new net: R21.2, R22.1, U7.7 (DIS)
- new net: D1.1 (K), R25.1
- new net: D5.1 (K), R28.1
- new net: R12.2, U3.10 (J), U3.11 (K)
- new net: R9.2, U2.5 (K), U2.6 (J)
- new net: R10.2, U2.10 (J), U2.11 (K)
- new net 555: SW4.2 (C), U7.3 (Q)
- new net Q0: D1.2 (A), U2.1 (Q), U2.13 (C), U4.7 (A)
- new net Q2: D3.2 (A), U3.1 (Q), U3.13 (C), U4.2 (C)
- no-connect marks 0 -> 6
Other:
- note added: "555 timer"
- note added: "JK bistabil"
- note added: "LED diode"
- note added: "Montažne rupe"
- note added: "Napajanje"
- note added: "Napajanje bistabila"
- note added: "Reset brojača"
- note added: "Tipkalo i ulaz radnog takta"
- moved on the sheet: C10, C6, R23, SW3, U6

Commit message: LV5
Parts:
- C2: renamed from C10; footprint (none) -> Capacitor_THT:CP_Radial_D5.0mm_P2.00mm; Manifacturer (none) -> SAMWHA; Part number (none) -> RD1A227M05011BB
- C3: renamed from C6; footprint (none) -> Capacitor_SMD:C_1206_3216Metric_Pad1.33x1.80mm_HandSolder; Manifacturer (none) -> SAMSUNG; Part number (none) -> CL31B105KBHNNNE
- C4: footprint (none) -> Capacitor_SMD:C_1206_3216Metric_Pad1.33x1.80mm_HandSolder; Manifacturer (none) -> SAMSUNG; Part number (none) -> CL31B104KBCNNNC
- C5: footprint (none) -> Capacitor_SMD:C_1206_3216Metric_Pad1.33x1.80mm_HandSolder; Manifacturer (none) -> SAMSUNG; Part number (none) -> CL31A106KBHNNNE
- D1, D2, D3, D5: footprint (none) -> LED_THT:LED_D5.0mm
- D4: Manifacturer part number (none) -> 11DQ06TA
- H1, H2, H3, H4: footprint (none) -> MountingHole:MountingHole_5.5mm
- L1: footprint (none) -> Inductor_THT:L_Radial_D7.2mm_P3.00mm_Murata_1700; Manifacturer (none) -> Inductor_THT:L_Radial_D7.2mm_P3.00mm_Murata_1700; Part number (none) -> COIL0608-0.33
- R1: renamed from R25; footprint (none) -> Resistor_THT:R_Axial_DIN0207_L6.3mm_D2.5mm_P10.16mm_Horizontal
- R10, R11, R12, R15, R9: footprint (none) -> Resistor_SMD:R_1206_3216Metric_Pad1.30x1.75mm_HandSolder
- R13: renamed from R23; footprint (none) -> Resistor_SMD:R_1206_3216Metric_Pad1.30x1.75mm_HandSolder; Manifacturer (none) -> ROYALOHM; Part number (none) -> 1206S4F2001T5E
- R14, R16, R17, R18, R6, R8: footprint (none) -> Resistor_SMD:R_1206_3216Metric_Pad1.30x1.75mm_HandSolder; Manifacturer (none) -> ROYALOHM
- R19: renamed from R21; footprint (none) -> Resistor_SMD:R_1206_3216Metric_Pad1.30x1.75mm_HandSolder; Manifacturer (none) -> ROYALOHM; Part number (none) -> 1206S4J0473T5E
- R2: renamed from R26; footprint (none) -> Resistor_THT:R_Axial_DIN0207_L6.3mm_D2.5mm_P10.16mm_Horizontal
- R20: renamed from R22; footprint (none) -> Resistor_SMD:R_1206_3216Metric_Pad1.30x1.75mm_HandSolder; Part number (none) -> 1206S4J0473T5E; manifacturer (none) -> ROYALOHM
- R3: renamed from R27; footprint (none) -> Resistor_THT:R_Axial_DIN0207_L6.3mm_D2.5mm_P10.16mm_Horizontal
- R4: renamed from R28; footprint (none) -> Resistor_THT:R_Axial_DIN0207_L6.3mm_D2.5mm_P10.16mm_Horizontal
- R5: footprint (none) -> Resistor_SMD:R_1206_3216Metric_Pad1.30x1.75mm_HandSolder; Manifacturer (none) -> ROYALOHM; Part number (none) -> 1206S4F2001T5E
- R7: renamed from R24; footprint (none) -> Resistor_SMD:R_1206_3216Metric_Pad1.30x1.75mm_HandSolder
- SW1: renamed from SW3; footprint (none) -> Button_Switch_THT:SW_PUSH_6mm_H4.3mm; Manifacturer (none) -> microswitch TACT; Part number (none) -> TACT-64N-F
- SW2: renamed from SW4; footprint (none) -> Button_Switch_THT:SW_Slide_SPDT_Straight_CK_OS102011MS2Q; Manifacturer (none) -> C&K; Part number (none) -> OS102011MS2QN1C
- U2: footprint (none) -> Package_DIP:DIP-16_W7.62mm_Socket_LongPads; manifacturer (none) -> RENESAS; part number (none) -> CD4027BMS
- U3: footprint (none) -> Package_DIP:DIP-16_W7.62mm_Socket_LongPads; Manifacturer (none) -> RENESAS; part number (none) -> CD4027BMS
- U4: footprint (none) -> Package_DIP:DIP-16_W7.62mm_Socket_LongPads; Manifacturer (none) -> TEXAS INSTRUMENTS; Part number (none) -> SN74LS47N
- U6: footprint (none) -> Package_TO_SOT_SMD:SOT-23-6; Manifacturer (none) -> TEXAS INSTRUMENTS; Part number (none) -> SN74LVC1G11DBVR
- U7: Manifacturere (none) -> TEXAS INSTRUMENTS; Part number (none) -> NE555P
