File: PTP_jakov_ozbolt_project-1/PTP_jakov_ozbolt_project-1.kicad_pcb (KiCad board)
At the start: 2 copper layers, 45 parts, among them U1 LM2574N-5, U2 4027, U3 4027, U4 74LS47, U5 HDSP-7401, U7 NE555P

Commit message: lv7
Parts:
- moved R6 158.2 mm to (190.9, 99.5)
- moved R5 158.1 mm to (190.9, 96.0)
- moved R8 157.4 mm to (191.0, 103.0)
- moved R16 147.8 mm to (191.0, 92.0)
- moved R9 129.9 mm to (161.2, 109.5), turned to 90 degrees
- moved R7 128.5 mm to (156.9, 109.5), turned to 90 degrees
- moved R20 93.4 mm to (114.2, 104.8), turned to 90 degrees
- moved R19 93.3 mm to (114.0, 98.0), turned to 90 degrees
- moved C5 83.9 mm to (131.0, 103.1), turned to -90 degrees
- moved C4 79.8 mm to (122.5, 110.0)
- moved R13 50.4 mm to (152.5, 109.5), turned to 90 degrees
- moved U6 48.3 mm to (139.4, 92.5)
- moved R10 43.3 mm to (165.5, 109.5), turned to 90 degrees
- moved R11 37.6 mm to (170.0, 109.5), turned to 90 degrees
- moved R12 32.4 mm to (174.0, 109.5), turned to 90 degrees
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Routing:
- net +5V: track 0.00 -> 227.4 mm, vias 0 -> 10
- net Net-(U7-THR): track 0.00 -> 91.3 mm, vias 0 -> 2
- net Net-(U7-DIS): track 0.00 -> 79.8 mm
- net Net-(D4-K): track 0.00 -> 70.2 mm
- net Q0: track 0.00 -> 67.2 mm, vias 0 -> 2
- net GND: track 0.00 -> 65.9 mm
- net Q3: track 0.00 -> 62.8 mm, vias 0 -> 6
- net Clock: track 0.00 -> 56.6 mm, vias 0 -> 2
- net Q1: track 0.00 -> 52.1 mm, vias 0 -> 3
- net VD: track 0.00 -> 48.5 mm
- net Reset: track 0.00 -> 35.8 mm, vias 0 -> 2
- net 555: track 0.00 -> 33.4 mm, vias 0 -> 2
- net Net-(SW2-A): track 0.00 -> 31.8 mm
- net Q2: track 0.00 -> 30.9 mm
- net Net-(U2A-J): track 0.00 -> 23.2 mm
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- added copper zone on B.Cu, net GND

Commit message: LV9
Other:
- board outline added: 100 x 80 mm
- board text added: "PTP - BCD counter Jakov Ožbolt"
